Commit message: Enhance diff_bot_sim with Gazebo simulation integration and improved URDF properties
- Updated docker-compose.yml for X server access and GPU capabilities
- Modified CMakeLists.txt to include worlds directory in installation
- Expanded diff_bot_display.launch.py to include Gazebo simulation launch
- Enhanced diff_bot.xacro with additional properties for chassis and wheels
- Added macros.xacro for inertia calculations
- Created empty.sdf for Gazebo world setup

File: src/diff_bot_sim/urdf/diff_bot.xacro (robot description, xacro)
@@ -1,9 +1,20 @@
 <?xml version="1.0"?>
 <robot name="diff_bot" xmlns:xacro="http://www.ros.org/wiki/xacro">
+    <!--................................ XACRO CONSTANTS .............................. -->
+    <xacro:property name="chassis_mass" value="70"/>
+    <xacro:property name="chassis_length" value="0.9"/>
+    <xacro:property name="chassis_width" value="0.64"/>
+    <xacro:property name="chassis_height" value="0.19"/>
+    <xacro:property name="traction_wheel_mass" value="1"/>
+    <xacro:property name="traction_wheel_radius" value="0.1"/>
+    <xacro:property name="traction_wheel_width" value="0.05"/>
+    <xacro:property name="traction_track_width" value="0.6"/>
+    <!-- ............................... LOAD MACROS ................................. -->
+    <xacro:include filename="$(find diff_bot_sim)/urdf/macros.xacro"/>
   <link name="world"/>
-  <link name="base_link">
+  <link name="chassis_link">
     <visual>
       <geometry>
-        <box size="0.9 0.64 0.19"/>
+        <box size="${chassis_length} ${chassis_width} ${chassis_height}"/>
       </geometry>
       <material name="grey">
@@ -11,9 +22,18 @@
       </material>
     </visual>
+    <collision>
+      <geometry>
+        <box size="${chassis_length} ${chassis_width} ${chassis_height}"/>
+      </geometry>
+    </collision>
+    <inertial>
+      <mass value="${chassis_mass}"/>
+      <xacro:box_inertia m="${chassis_mass}" x="${chassis_length}" y="${chassis_width}" z = "${chassis_height}"/>
+    </inertial>
   </link>
   <link name="left_wheel">
     <visual>
       <geometry>
-        <cylinder radius="0.13" length="0.05"/>
+        <cylinder radius="${traction_wheel_radius}" length="${traction_wheel_width}"/>
       </geometry>
       <material name="black">
@@ -21,9 +41,19 @@
       </material>
     </visual>
+    <collision>
+      <geometry>
+        <cylinder radius="${traction_wheel_radius}" length="${traction_wheel_width}"/>
+      </geometry>
+    </collision>
+    <inertial>
+        <origin xyz="0 0 0" rpy="0 ${pi/2} ${pi/2}" />
+        <mass value="${traction_wheel_mass}"/>
+        <xacro:cylinder_inertia m="${traction_wheel_mass}" r="${traction_wheel_radius}" h="${traction_wheel_width}"/>
+    </inertial>
   </link>
   <link name="right_wheel">
     <visual>
       <geometry>
-        <cylinder radius="0.13" length="0.05"/>
+        <cylinder radius="${traction_wheel_radius}" length="${traction_wheel_width}"/>
       </geometry>
       <material name="black">
@@ -31,4 +61,14 @@
       </material>
     </visual>
+    <collision>
+      <geometry>
+        <cylinder radius="${traction_wheel_radius}" length="${traction_wheel_width}"/>
+      </geometry>
+    </collision>
+    <inertial>
+        <origin xyz="0 0 0" rpy="0 ${pi/2} ${pi/2}" />
+        <mass value="${traction_wheel_mass}"/>
+        <xacro:cylinder_inertia m="${traction_wheel_mass}" r="${traction_wheel_radius}" h="${traction_wheel_width}"/>
+    </inertial>
   </link>
   <link name="caster_wheel">
@@ -41,12 +81,21 @@
       </material>
     </visual>
+    <collision>
+      <geometry>
+        <sphere radius="0.1"/>
+      </geometry>
+    </collision>
+    <inertial>
+        <mass value="0.5"/>
+        <xacro:sphere_inertia m="0.5" r="0.1"/>
+    </inertial>
   </link>
-  <joint name="world_to_base_link" type="fixed">
+  <joint name="world_to_chassis_link" type="fixed">
     <parent link="world"/>
-    <child link="base_link"/>
+    <child link="chassis_link"/>
     <origin xyz="0 0 0" rpy="0 0 0"/>
   </joint>
   <joint name="left_wheel_joint" type="continuous">
-    <parent link="base_link"/>
+    <parent link="chassis_link"/>
     <child link="left_wheel"/>
     <origin xyz="0.25 0.35 -0.12" rpy="1.57 0 0"/>
@@ -54,5 +103,5 @@
   </joint>
   <joint name="right_wheel_joint" type="continuous">
-    <parent link="base_link"/>
+    <parent link="chassis_link"/>
     <child link="right_wheel"/>
     <origin xyz="0.25 -0.35 -0.12" rpy="1.57 0 0"/>
@@ -60,5 +109,5 @@
   </joint>
   <joint name="caster_wheel_joint" type="fixed">
-    <parent link="base_link"/>
+    <parent link="chassis_link"/>
     <child link="caster_wheel"/>
     <origin xyz="-0.35 0 -0.12" rpy="0 0 0"/>

Commit message: Refactor diff_bot launch files for improved simulation support and update URDF structure

File: src/diff_bot_sim/urdf/diff_bot.xacro (robot description, xacro)
@@ -10,7 +10,10 @@
     <xacro:property name="traction_wheel_width" value="0.05"/>
     <xacro:property name="traction_track_width" value="0.6"/>
-    <!-- ............................... LOAD MACROS ................................. -->
-    <xacro:include filename="$(find diff_bot_sim)/urdf/macros.xacro"/>
-  <link name="world"/>
+    <xacro:arg name="sim_ign" default="true" />
+  <xacro:if value="$(arg sim_ign)">
+      <xacro:include filename="$(find diff_bot_sim)/urdf/ign.xacro"/>
+  </xacro:if>
+  <xacro:include filename="$(find diff_bot_sim)/urdf/macros.xacro"/>
+  <link name="base_link"/>
   <link name="chassis_link">
     <visual>
@@ -91,6 +94,6 @@
     </inertial>
   </link>
-  <joint name="world_to_chassis_link" type="fixed">
-    <parent link="world"/>
+  <joint name="chassis_joint" type="fixed">
+    <parent link="base_link"/>
     <child link="chassis_link"/>
     <origin xyz="0 0 0" rpy="0 0 0"/>

Commit message: Update Dockerfile and URDF files for diff_bot simulation enhancements
- Replace teleop-twist-joy with turtlesim in Dockerfile dependencies
- Add cmd_vel remapping in diff_bot_ign.launch.py
- Introduce caster wheel links and joints in diff_bot.xacro
- Implement DiffDrive plugin in ign.xacro for improved drive control

File: src/diff_bot_sim/urdf/diff_bot.xacro (robot description, xacro)
@@ -54,4 +54,5 @@
         <xacro:cylinder_inertia m="${traction_wheel_mass}" r="${traction_wheel_radius}" h="${traction_wheel_width}"/>
     </inertial>
+    <mu>5.0</mu>
   </link>
   <link name="right_wheel">
@@ -74,6 +75,7 @@
         <xacro:cylinder_inertia m="${traction_wheel_mass}" r="${traction_wheel_radius}" h="${traction_wheel_width}"/>
     </inertial>
+    <mu>5.0</mu>
   </link>
-  <link name="caster_wheel">
+  <link name="caster_wheel_front">
     <visual>
       <geometry>
@@ -93,4 +95,25 @@
         <xacro:sphere_inertia m="0.5" r="0.1"/>
     </inertial>
+    <mu>0.0</mu>
+  </link>
+  <link name="caster_wheel_back">
+    <visual>
+      <geometry>
+        <sphere radius="0.1"/>
+      </geometry>
+      <material name="black">
+        <color rgba="0.0 0.0 0.0 1.0"/>
+      </material>
+    </visual>
+    <collision>
+      <geometry>
+        <sphere radius="0.1"/>
+      </geometry>
+    </collision>
+    <inertial>
+        <mass value="0.5"/>
+        <xacro:sphere_inertia m="0.5" r="0.1"/>
+    </inertial>
+    <mu>0.0</mu>
   </link>
   <joint name="chassis_joint" type="fixed">
@@ -102,17 +125,22 @@
     <parent link="chassis_link"/>
     <child link="left_wheel"/>
-    <origin xyz="0.25 0.35 -0.12" rpy="1.57 0 0"/>
-    <axis xyz="0 1 0"/>
+    <origin xyz="0.0 0.35 -0.12" rpy="1.57 0 0"/>
+    <axis xyz="0 0 1"/>
   </joint>
   <joint name="right_wheel_joint" type="continuous">
     <parent link="chassis_link"/>
     <child link="right_wheel"/>
-    <origin xyz="0.25 -0.35 -0.12" rpy="1.57 0 0"/>
-    <axis xyz="0 1 0"/>
+    <origin xyz="0.0 -0.35 -0.12" rpy="1.57 0 0"/>
+    <axis xyz="0 0 1"/>
   </joint>
-  <joint name="caster_wheel_joint" type="fixed">
+  <joint name="caster_wheel_front_joint" type="fixed">
     <parent link="chassis_link"/>
-    <child link="caster_wheel"/>
+    <child link="caster_wheel_front"/>
     <origin xyz="-0.35 0 -0.12" rpy="0 0 0"/>
   </joint>
+  <joint name="caster_wheel_back_joint" type="fixed">
+    <parent link="chassis_link"/>
+    <child link="caster_wheel_back"/>
+    <origin xyz="0.35 0 -0.12" rpy="0 0 0"/>
+  </joint>
 </robot>

File: src/diff_bot_sim/urdf/ign.xacro (robot description, xacro)
@@ -6,8 +6,18 @@
             <render_engine>ogre2</render_engine>
         </plugin>
-        <!-- <plugin filename="ignition-gazebo-imu-system" name="ignition::gazebo::systems::Imu">
-        </plugin> -->
         <plugin filename="ignition-gazebo-joint-state-publisher-system" name="ignition::gazebo::systems::JointStatePublisher">
         </plugin>
     </gazebo>
+    <gazebo>
+        <plugin
+            filename="libignition-gazebo-diff-drive-system.so"
+            name="ignition::gazebo::systems::DiffDrive">
+            <left_joint>left_wheel_joint</left_joint>
+            <right_joint>right_wheel_joint</right_joint>
+            <wheel_separation>0.7</wheel_separation>
+            <wheel_radius>0.1</wheel_radius>
+            <odom_publish_frequency>1</odom_publish_frequency>
+            <topic>cmd_vel</topic>
+        </plugin>
+    </gazebo>
 </robot>

Commit message: Add 2D LIDAR support to diff_bot simulation with updated URDF and launch files

File: src/diff_bot_sim/urdf/diff_bot.xacro (robot description, xacro)
@@ -10,4 +10,10 @@
     <xacro:property name="traction_wheel_width" value="0.05"/>
     <xacro:property name="traction_track_width" value="0.6"/>
+    <xacro:property name="two_d_lidar_update_rate" value="30"/>
+    <xacro:property name="two_d_lidar_sample_size" value="361"/>
+    <xacro:property name="two_d_lidar_min_angle" value="0"/>
+    <xacro:property name="two_d_lidar_max_angle" value="360"/>
+    <xacro:property name="two_d_lidar_min_range" value="0.55"/>
+    <xacro:property name="two_d_lidar_max_range" value="16"/>
     <xacro:arg name="sim_ign" default="true" />
   <xacro:if value="$(arg sim_ign)">
@@ -125,5 +131,5 @@
     <parent link="chassis_link"/>
     <child link="left_wheel"/>
-    <origin xyz="0.0 0.35 -0.12" rpy="1.57 0 0"/>
+    <origin xyz="0.0 0.35 -0.12" rpy="-1.57 0 0"/>
     <axis xyz="0 0 1"/>
   </joint>
@@ -131,5 +137,5 @@
     <parent link="chassis_link"/>
     <child link="right_wheel"/>
-    <origin xyz="0.0 -0.35 -0.12" rpy="1.57 0 0"/>
+    <origin xyz="0.0 -0.35 -0.12" rpy="-1.57 0 0"/>
     <axis xyz="0 0 1"/>
   </joint>
@@ -137,10 +143,35 @@
     <parent link="chassis_link"/>
     <child link="caster_wheel_front"/>
-    <origin xyz="-0.35 0 -0.12" rpy="0 0 0"/>
+    <origin xyz="0.35 0 -0.12" rpy="0 0 0"/>
   </joint>
   <joint name="caster_wheel_back_joint" type="fixed">
     <parent link="chassis_link"/>
     <child link="caster_wheel_back"/>
-    <origin xyz="0.35 0 -0.12" rpy="0 0 0"/>
+    <origin xyz="-0.35 0 -0.12" rpy="0 0 0"/>
+  </joint>
+    <!--................................ LIDAR .............................. -->
+  <link name="two_d_lidar">
+    <visual>
+      <geometry>
+        <cylinder radius="0.07" length="0.05"/>
+      </geometry>
+      <material name="black">
+        <color rgba="0.0 0.0 0.0 1.0"/>
+      </material>
+    </visual>
+    <collision>
+      <geometry>
+        <cylinder radius="0.07" length="0.05"/>
+      </geometry>
+    </collision>
+    <inertial>
+        <mass value="0.5"/>
+        <xacro:cylinder_inertia m="0.5" r="0.07" h="0.05"/>
+    </inertial>
+  </link>
+  <joint name="lidar_joint" type="fixed">
+    <parent link="chassis_link"/>
+    <child link="two_d_lidar"/>
+    <origin xyz="0.1 0 0.12" rpy="0 0 0"/>
   </joint>
 </robot>

File: src/diff_bot_sim/urdf/ign.xacro (robot description, xacro)
@@ -21,3 +21,32 @@
         </plugin>
     </gazebo>
+    <gazebo reference="two_d_lidar">
+        <sensor name='gpu_lidar' type='gpu_lidar'>
+            <topic>scan</topic>
+            <update_rate>${two_d_lidar_update_rate}</update_rate>
+            <ignition_frame_id>two_d_lidar</ignition_frame_id>
+            <lidar>
+                <scan>
+                    <horizontal>
+                        <samples>${two_d_lidar_sample_size}</samples>
+                        <resolution>1</resolution>
+                        <min_angle>${radians(two_d_lidar_min_angle)}</min_angle>
+                        <max_angle>${radians(two_d_lidar_max_angle)}</max_angle>
+                    </horizontal>
+                </scan>
+                <range>
+                    <min>${two_d_lidar_min_range}</min>
+                    <max>${two_d_lidar_max_range}</max>
+                    <resolution>0.01</resolution>
+                </range>
+                <noise>
+                    <type>gaussian</type>
+                    <mean>0.0</mean>
+                    <stddev>0.001</stddev>
+                </noise>
+            </lidar>
+            <alwaysOn>1</alwaysOn>
+            <visualize>true</visualize>
+        </sensor>
+    </gazebo>
 </robot>
